File: gauge.kicad_pcb (KiCad board)
At the start: 2 copper layers, 200 x 35 mm, 17 parts, among them J1 8P8C_LED_Shielded, J10 Conn_01x08_Male, J11 Conn_01x09_Male, J12 Conn_01x06_Male, J13 Conn_01x10_Male, J15 Conn_01x18_Male, J2 USB_A, J3 USB_B_Micro, J4 Conn_01x06_Male, J6 USB_A, J7 Conn_01x06_Male, J8 Conn_01x13_Male, J9 Conn_01x06_Male, U1 W25Q128JVS, U2 W25Q32JVZP, U3 WM8731CLSEFL

Commit message: the ruler V2! Now better, stronger, faster
Parts:
- removed D1: APA102-2020, LED_SMD:LED-APA102-2020
- removed J11: Conn_01x09_Male, Connector_PinHeader_2.54mm:PinHeader_1x09_P2.54mm_Vertical
- removed J12: Conn_01x06_Male, Connector_PinHeader_2.54mm:PinHeader_1x06_P2.54mm_Vertical
- removed J13: Conn_01x10_Male, Connector_PinHeader_2.54mm:PinHeader_1x10_P2.54mm_Vertical
- removed J15: Conn_01x18_Male, Connector_PinHeader_2.54mm:PinHeader_1x18_P2.54mm_Vertical
- removed U3: WM8731CLSEFL, Package_DFN_QFN:QFN-28-1EP_5x5mm_P0.5mm_EP3.35x3.35mm
- added C1: C_Polarized_Small, Capacitor_THT:CP_Radial_D4.0mm_P1.50mm, F.Cu at (68.5, 91.5)
- added C2: C_Polarized_Small, Capacitor_THT:CP_Radial_D4.0mm_P1.50mm, F.Cu at (75.0, 91.5)
- added C3: 22nF, Capacitor_THT:CP_Radial_D4.0mm_P1.50mm, F.Cu at (37.2, 92.0)
- added C4: 22nF, Capacitor_THT:CP_Radial_D4.0mm_P1.50mm, F.Cu at (49.5, 102.5)
- added J5: AudioJack3, Connector_Audio:Jack_3.5mm_CUI_SJ-3523-SMT_Horizontal, F.Cu at (193.5, 114.0)
- added JP1: SolderJumper_2_Open, Jumper:SolderJumper-2_P1.3mm_Open_Pad1.0x1.5mm, F.Cu at (110.2, 96.5)
- added JP10: SolderJumper_2_Open, Jumper:SolderJumper-2_P1.3mm_Open_Pad1.0x1.5mm, F.Cu at (187.0, 101.5)
- added JP11: SolderJumper_2_Open, Jumper:SolderJumper-2_P1.3mm_Open_Pad1.0x1.5mm, F.Cu at (190.6, 101.5)
- added JP12: SolderJumper_2_Open, Jumper:SolderJumper-2_P1.3mm_Open_Pad1.0x1.5mm, F.Cu at (194.1, 101.5)
- added JP13: SolderJumper_2_Open, Jumper:SolderJumper-2_P1.3mm_Open_Pad1.0x1.5mm, F.Cu at (197.7, 101.5)
- added JP14: SolderJumper_2_Open, Jumper:SolderJumper-2_P1.3mm_Open_Pad1.0x1.5mm, F.Cu at (156.3, 109.0)
- added JP15: SolderJumper_2_Open, Jumper:SolderJumper-2_P1.3mm_Open_Pad1.0x1.5mm, F.Cu at (156.3, 106.0)
- added JP16: SolderJumper_2_Open, Jumper:SolderJumper-2_P1.3mm_Open_Pad1.0x1.5mm, F.Cu at (156.3, 103.0)
- added JP17: SolderJumper_2_Open, Jumper:SolderJumper-2_P1.3mm_Open_Pad1.0x1.5mm, F.Cu at (156.3, 100.0)
- added JP18: 3.3v, Jumper:SolderJumper-2_P1.3mm_Open_Pad1.0x1.5mm, F.Cu at (59.0, 103.7)
- added JP19: 5v, Jumper:SolderJumper-2_P1.3mm_Open_Pad1.0x1.5mm, F.Cu at (59.0, 100.1)
- added JP2: SolderJumper_2_Open, Jumper:SolderJumper-2_P1.3mm_Open_Pad1.0x1.5mm, F.Cu at (106.7, 96.5)
- added JP20: 3.3v, Jumper:SolderJumper-2_P1.3mm_Open_Pad1.0x1.5mm, F.Cu at (47.0, 95.7)
- added JP21: 5v, Jumper:SolderJumper-2_P1.3mm_Open_Pad1.0x1.5mm, F.Cu at (47.0, 92.2)
- added JP22: SolderJumper_2_Open, Jumper:SolderJumper-2_P1.3mm_Open_Pad1.0x1.5mm, F.Cu at (95.0, 111.5)
- added JP23: SolderJumper_2_Open, Jumper:SolderJumper-2_P1.3mm_Open_Pad1.0x1.5mm, F.Cu at (97.9, 111.5)
- added JP24: SolderJumper_2_Open, Jumper:SolderJumper-2_P1.3mm_Open_Pad1.0x1.5mm, F.Cu at (101.0, 111.5)
- added JP25: SolderJumper_2_Open, Jumper:SolderJumper-2_P1.3mm_Open_Pad1.0x1.5mm, F.Cu at (104.0, 111.5)
- added JP26: 3.3v, Jumper:SolderJumper-2_P1.3mm_Open_Pad1.0x1.5mm, F.Cu at (86.3, 117.5)
- added JP27: 5v, Jumper:SolderJumper-2_P1.3mm_Open_Pad1.0x1.5mm, F.Cu at (89.9, 117.5)
- added JP3: SolderJumper_2_Open, Jumper:SolderJumper-2_P1.3mm_Open_Pad1.0x1.5mm, F.Cu at (103.1, 96.5)
- added JP4: SolderJumper_2_Open, Jumper:SolderJumper-2_P1.3mm_Open_Pad1.0x1.5mm, F.Cu at (99.5, 96.5)
- added JP5: SolderJumper_2_Open, Jumper:SolderJumper-2_P1.3mm_Open_Pad1.0x1.5mm, F.Cu at (96.0, 96.5)
- added JP6: 3.3v, Jumper:SolderJumper-2_P1.3mm_Open_Pad1.0x1.5mm, F.Cu at (70.5, 96.7)
- added JP7: 5v, Jumper:SolderJumper-2_P1.3mm_Open_Pad1.0x1.5mm, F.Cu at (74.0, 96.7)
- added JP8: SolderJumper_2_Open, Jumper:SolderJumper-2_P1.3mm_Open_Pad1.0x1.5mm, F.Cu at (179.9, 101.5)
- added JP9: SolderJumper_2_Open, Jumper:SolderJumper-2_P1.3mm_Open_Pad1.0x1.5mm, F.Cu at (183.4, 101.5)
- added OA1: TLV2371P, Package_DIP:DIP-8_W7.62mm, F.Cu at (48.2, 109.2)
- added OA2: TLV2371D, Package_SO:SOIC-8_3.9x4.9mm_P1.27mm, F.Cu at (41.0, 100.0)
- J1: value 8P8C_LED_Shielded -> pin offset +8; footprint Connector_RJ:RJ45_Amphenol_RJMG1BD3B8K1ANR -> Connector_PinHeader_2.54mm:PinHeader_1x05_P2.54mm_Vertical
- J10: value Conn_01x08_Male -> pin offset +1; footprint Connector_PinHeader_2.54mm:PinHeader_1x08_P2.54mm_Vertical -> Connector_PinHeader_2.54mm:PinHeader_1x05_P2.54mm_Vertical
- J2: value USB_A -> power; footprint Connector_USB:USB_A_CNCTech_1001-011-01101_Horizontal -> Connector_PinHeader_2.54mm:PinHeader_1x05_P2.54mm_Vertical
- J3: value USB_B_Micro -> pin offset +25; footprint Connector_USB:USB_Micro-AB_Molex_47590-0001 -> Connector_PinHeader_2.54mm:PinHeader_1x04_P2.54mm_Vertical
- J4: value Conn_01x06_Male -> pin offset +13; footprint Connector_PinHeader_2.54mm:PinHeader_1x06_P2.54mm_Vertical -> Connector_PinHeader_2.54mm:PinHeader_1x02_P2.54mm_Vertical
- J6: value USB_A -> Jack-DC; footprint Connector_USB:USB_A_Molex_67643_Horizontal -> Connector_BarrelJack:BarrelJack_SwitchcraftConxall_RAPC10U_Horizontal
- J7: value Conn_01x06_Male -> AudioJack3; footprint Connector_PinHeader_2.54mm:PinHeader_1x06_P2.54mm_Vertical -> Connector_Audio:Jack_3.5mm_CUI_SJ-3523-SMT_Horizontal
- J8: value Conn_01x13_Male -> OA1_out; footprint Connector_PinHeader_2.54mm:PinHeader_1x13_P2.54mm_Vertical -> Connector_PinHeader_2.54mm:PinHeader_1x02_P2.54mm_Vertical
- J9: value Conn_01x06_Male -> OA2_out; footprint Connector_PinHeader_2.54mm:PinHeader_1x06_P2.54mm_Vertical -> Connector_PinHeader_2.54mm:PinHeader_1x02_P2.54mm_Vertical
- U1: value W25Q128JVS -> rp2040-zero-pads; footprint Package_SO:SOIC-8_5.23x5.23mm_P1.27mm -> kleeb:rp2040-zero-tht-pads-cutout
- U2: value W25Q32JVZP -> W25Q32JVSS; footprint Package_SON:WSON-8-1EP_6x5mm_P1.27mm_EP3.4x4.3mm -> Package_SO:SOIC-8_5.23x5.23mm_P1.27mm
- moved J2 118.6 mm to (157.5, 117.5), turned to 90 degrees
- moved J8 113.1 mm to (33.0, 114.8), turned to 180 degrees
- moved J7 107.8 mm to (181.5, 114.0), turned to 180 degrees
- moved U2 76.1 mm to (113.5, 110.5), turned to 90 degrees
- moved J3 72.9 mm to (169.7, 99.9)
- moved J1 59.1 mm to (108.0, 92.0), turned to -90 degrees
- moved J10 53.6 mm to (104.5, 116.5), turned to -90 degrees
- moved U1 35.9 mm to (131.0, 107.5), turned to 180 degrees
- moved J4 18.6 mm to (145.0, 97.0), turned to 0 degrees
- moved J9 14.8 mm to (33.0, 100.5), turned to 180 degrees
- moved J6 8.04 mm to (70.5, 101.3), turned to 90 degrees
Connections:
- J10 pad 1: Net-(U1-Pad1) -> Net-(J10-Pin_1)
- J10 pad 2: Net-(U1-Pad2) -> Net-(J10-Pin_2)
- J10 pad 3: Net-(U1-Pad3) -> Net-(J10-Pin_3)
- J10 pad 4: Net-(U1-Pad4) -> Net-(J10-Pin_4)
- J10 pad 5: Net-(U1-Pad5) -> Net-(J10-Pin_5)
- J2 pad 1: Net-(J2-Pad1) -> +5V
- J2 pad 2: Net-(J2-Pad2) -> unconnected-(J2-Pin_2-Pad2)
- J2 pad 3: Net-(J2-Pad3) -> GND
- J2 pad 4: Net-(J2-Pad4) -> unconnected-(J2-Pin_4-Pad4)
- J2 pad 5: Net-(J2-Pad5) -> +3.3V
- J4 pad 1: Net-(D1-Pad1) -> Net-(J4-Pin_1)
- J4 pad 2: Net-(D1-Pad2) -> Net-(J4-Pin_2)
- J6 pad 1: Net-(J6-Pad1) -> Net-(JP6-A)
- J6 pad 2: Net-(J7-Pad2) -> GND
- J8 pad 2: Net-(J1-Pad2) -> GND
- J9 pad 1: Net-(J2-Pad1) -> Net-(J9-Pin_1)
- J9 pad 2: Net-(J2-Pad2) -> GND
- U1 pad 1: Net-(U1-Pad1) -> unconnected-(U1-0-Pad1)
- U1 pad 2: Net-(U1-Pad2) -> unconnected-(U1-1-Pad2)
- U1 pad 3: Net-(U1-Pad3) -> Net-(JP25-B)
- U1 pad 4: Net-(U1-Pad4) -> Net-(JP24-B)
- U1 pad 5: Net-(U1-Pad5) -> Net-(JP23-B)
- U1 pad 6: Net-(U1-Pad6) -> Net-(JP22-B)
- U1 pad 7: Net-(U1-Pad7) -> unconnected-(U1-6-Pad7)
- U1 pad 8: Net-(U1-Pad8) -> unconnected-(U1-7-Pad8)
- U2 pad 1: Net-(U2-Pad1) -> Net-(JP22-B)
- U2 pad 2: Net-(U2-Pad2) -> Net-(JP24-B)
- U2 pad 3: Net-(U2-Pad3) -> unconnected-(U2-IO2-Pad3)
- U2 pad 4: Net-(U2-Pad4) -> GND
- U2 pad 5: Net-(U2-Pad5) -> Net-(JP23-B)
- U2 pad 6: Net-(U2-Pad6) -> Net-(JP25-B)
- U2 pad 7: Net-(U2-Pad7) -> unconnected-(U2-IO3-Pad7)
- U2 pad 8: Net-(U2-Pad8) -> +3.3V
Routing:
- net +3.3V: track 0.00 -> 245.6 mm, vias 0 -> 4
- net +5V: track 0.00 -> 238.0 mm, vias 0 -> 3
- net Net-(JP4-B): track 0.00 -> 125.2 mm, vias 0 -> 1
- net Net-(JP5-B): track 0.00 -> 122.9 mm, vias 0 -> 1
- net Net-(U3-Pad28): track 116.7 -> 0.00 mm, vias 2 -> 0
- net Net-(U3-Pad27): track 114.5 -> 0.00 mm, vias 2 -> 0
- net GND: track 0.00 -> 95.3 mm, vias 0 -> 9
- net Net-(U3-Pad25): track 77.4 -> 0.00 mm, vias 1 -> 0
- net Net-(U3-Pad26): track 76.1 -> 0.00 mm, vias 1 -> 0
- net Net-(U3-Pad3): track 66.9 -> 0.00 mm, vias 1 -> 0
- net Net-(JP11-B): track 0.00 -> 66.6 mm, vias 0 -> 2
- net Net-(U3-Pad5): track 62.0 -> 0.00 mm, vias 1 -> 0
- net Net-(U3-Pad15): track 60.5 -> 0.00 mm, vias 1 -> 0
- net Net-(JP10-B): track 0.00 -> 58.7 mm, vias 0 -> 2
- net Net-(JP16-A): track 0.00 -> 56.3 mm, vias 0 -> 2
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- added copper zone on B.Cu, net GND
- added copper zone on F.Cu, net GND
Other:
- board size 200 x 35 mm -> 200 x 35.5 mm
- board text added: "vega76.cz"
- board text removed: "Electrical engineers do work with more frequency and less resistance"
- board text removed: "Information theory began as a bridge from mathematics to electrical engineering and from there to computing."
- board text removed: "Neon signs don't consume much power, but they look like they do. A cousin of fluorescent lighting, neon is actually quite energy efficient. A neon tube glows coolly when high-voltage, low-amperage electrical power excites the gas within it."
- board text removed: "THE RULER"
- board text removed: "art without engineering is dreaming, engineering without art is calculating"
- board text removed: "designed by @vega_D"
- board text removed: "ethernet"
- board text removed: "flash"
- board text removed: "flash 2"
- board text removed: "not tm"
- board text removed: "one person's magic is another's engineering"
- board text removed: "qfn 28"
- board text removed: "rgb led"
- board text removed: "usb a plug"
- board text removed: "usb a port"
- board text removed: "usb b micro port"
- board text removed: "while it is convinient to think that energy flows over wires, it's actually transmitted over the field."
