File: gauge.kicad_sch (KiCad schematic)
At the start: 17 parts, among them J1 8P8C_LED_Shielded, J10 Conn_01x08_Male, J11 Conn_01x09_Male, J12 Conn_01x06_Male, J13 Conn_01x10_Male, J15 Conn_01x18_Male, J2 USB_A, J3 USB_B_Micro, J4 Conn_01x06_Male, J6 USB_A, J7 Conn_01x06_Male, J8 Conn_01x13_Male, J9 Conn_01x06_Male, U1 W25Q128JVS, U2 W25Q32JVZP, U3 WM8731CLSEFL

Commit message: the ruler V2! Now better, stronger, faster
Parts:
- removed D1: APA102-2020, LED_SMD:LED-APA102-2020, symbol LED:APA102-2020
- removed J1: 8P8C_LED_Shielded, Connector_RJ:RJ45_Amphenol_RJMG1BD3B8K1ANR, symbol Connector:8P8C_LED_Shielded
- removed J10: Conn_01x08_Male, Connector_PinHeader_2.54mm:PinHeader_1x08_P2.54mm_Vertical, symbol Connector:Conn_01x08_Male
- removed J11: Conn_01x09_Male, Connector_PinHeader_2.54mm:PinHeader_1x09_P2.54mm_Vertical, symbol Connector:Conn_01x09_Male
- removed J12, J4, J7, J9: Conn_01x06_Male, Connector_PinHeader_2.54mm:PinHeader_1x06_P2.54mm_Vertical, symbol Connector:Conn_01x06_Male
- removed J13: Conn_01x10_Male, Connector_PinHeader_2.54mm:PinHeader_1x10_P2.54mm_Vertical, symbol Connector:Conn_01x10_Male
- removed J15: Conn_01x18_Male, Connector_PinHeader_2.54mm:PinHeader_1x18_P2.54mm_Vertical, symbol Connector:Conn_01x18_Male
- removed J2: USB_A, Connector_USB:USB_A_CNCTech_1001-011-01101_Horizontal, symbol Connector:USB_A
- removed J3: USB_B_Micro, Connector_USB:USB_Micro-AB_Molex_47590-0001, symbol Connector:USB_B_Micro
- removed J6: USB_A, Connector_USB:USB_A_Molex_67643_Horizontal, symbol Connector:USB_A
- removed J8: Conn_01x13_Male, Connector_PinHeader_2.54mm:PinHeader_1x13_P2.54mm_Vertical, symbol Connector:Conn_01x13_Male
- removed U1: W25Q128JVS, Package_SO:SOIC-8_5.23x5.23mm_P1.27mm, symbol Memory_Flash:W25Q128JVS
- removed U2: W25Q32JVZP, Package_SON:WSON-8-1EP_6x5mm_P1.27mm_EP3.4x4.3mm, symbol Memory_Flash:W25Q32JVZP
- removed U3: WM8731CLSEFL, Package_DFN_QFN:QFN-28-1EP_5x5mm_P0.5mm_EP3.35x3.35mm, symbol Audio:WM8731CLSEFL
- added C1, C2: C_Polarized_Small, Capacitor_THT:CP_Radial_D4.0mm_P1.50mm, symbol Device:C_Polarized_Small
- added C3, C4: 22nF, Capacitor_THT:CP_Radial_D4.0mm_P1.50mm, symbol Device:C_Polarized_Small
- added J1: pin offset +8, Connector_PinHeader_2.54mm:PinHeader_1x05_P2.54mm_Vertical, symbol Connector:Conn_01x05_Pin
- added J10: pin offset +1, Connector_PinHeader_2.54mm:PinHeader_1x05_P2.54mm_Vertical, symbol Connector:Conn_01x05_Pin
- added J2: power, Connector_PinHeader_2.54mm:PinHeader_1x05_P2.54mm_Vertical, symbol Connector:Conn_01x05_Pin
- added J3: pin offset +25, Connector_PinHeader_2.54mm:PinHeader_1x04_P2.54mm_Vertical, symbol Connector:Conn_01x04_Pin
- added J4: pin offset +13, Connector_PinHeader_2.54mm:PinHeader_1x02_P2.54mm_Vertical, symbol Connector:Conn_01x02_Pin
- added J5, J7: AudioJack3, Connector_Audio:Jack_3.5mm_CUI_SJ-3523-SMT_Horizontal, symbol Connector_Audio:AudioJack3
- added J6: Jack-DC, Connector_BarrelJack:BarrelJack_SwitchcraftConxall_RAPC10U_Horizontal, symbol Connector:Jack-DC
- added J8: OA1_out, Connector_PinHeader_2.54mm:PinHeader_1x02_P2.54mm_Vertical, symbol Connector:Conn_01x02_Pin
- added J9: OA2_out, Connector_PinHeader_2.54mm:PinHeader_1x02_P2.54mm_Vertical, symbol Connector:Conn_01x02_Pin
- added JP1, JP10, JP11, JP12, JP13, JP14, JP15, JP16, JP17, JP2, JP22, JP23, JP24, JP25, JP3, JP4, JP5, JP8, JP9: SolderJumper_2_Open, Jumper:SolderJumper-2_P1.3mm_Open_Pad1.0x1.5mm, symbol Jumper:SolderJumper_2_Open
- added JP18, JP20, JP26, JP6: 3.3v, Jumper:SolderJumper-2_P1.3mm_Open_Pad1.0x1.5mm, symbol Jumper:SolderJumper_2_Open
- added JP19, JP21, JP27, JP7: 5v, Jumper:SolderJumper-2_P1.3mm_Open_Pad1.0x1.5mm, symbol Jumper:SolderJumper_2_Open
- added OA1: TLV2371P, Package_DIP:DIP-8_W7.62mm, symbol Amplifier_Operational:TLV2371P
- added OA2: TLV2371D, Package_SO:SOIC-8_3.9x4.9mm_P1.27mm, symbol Amplifier_Operational:TLV2371D
- added U1: rp2040-zero-pads, kleeb:rp2040-zero-tht-pads-cutout, symbol mcu:rp2040-zero-pads
- added U2: W25Q32JVSS, Package_SO:SOIC-8_5.23x5.23mm_P1.27mm, symbol Memory_Flash:W25Q32JVSS
Connections:
- new net: J5.R, JP10.1 (A)
- new net: J5.S, JP13.1 (A)
- new net: J5.T, JP11.1 (A)
- new net: J10.3 (Pin_3), JP23.1 (A)
- new net: JP23.2 (B), U1.5 (4), U2.5 (DI(IO0))
- new net: J1.2 (Pin_2), JP2.1 (A)
- new net: JP2.2 (B), U1.11 (10)
- new net: J1.3 (Pin_3), JP3.1 (A)
- new net: JP3.2 (B), U1.12 (11)
- new net: JP20.1 (A), JP21.2 (B), OA2.7 (V+)
- new net: J1.5 (Pin_5), JP5.1 (A)
- new net: C3.1, JP5.2 (B), OA2.3 (+), U1.14 (13)
- new net: J6.1, JP6.1 (A), JP7.2 (B)
- new net: J10.1 (Pin_1), JP25.1 (A)
- new net: JP25.2 (B), U1.3 (2), U2.6 (CLK)
- new net: JP16.1 (A), JP9.2 (B), U1.18 (27)
- new net: J3.2 (Pin_2), JP16.2 (B)
- new net: J8.1 (Pin_1), OA1.2 (-), OA1.6
- new net: C4.1, JP4.2 (B), OA1.3 (+), U1.13 (12)
- new net: JP18.1 (A), JP19.2 (B), OA1.7 (V+)
- new net: JP10.2 (B), JP15.1 (A), U1.19 (28)
- new net: J1.1 (Pin_1), JP1.1 (A)
- new net: J1.4 (Pin_4), JP4.1 (A)
- new net: JP1.2 (B), U1.10 (9)
- new net: J4.1 (Pin_1), U1.15 (14)
- new net: J4.2 (Pin_2), U1.16 (15)
- new net: JP17.1 (A), JP8.2 (B), U1.17 (26)
- new net: JP11.2 (B), JP14.1 (A), U1.20 (29)
- new net: JP24.2 (B), U1.4 (3), U2.2 (DO(IO1))
- new net: JP22.2 (B), U1.6 (5), U2.1 (~{CS})
- new net: J7.T, JP9.1 (A)
- new net: J3.4 (Pin_4), JP14.2 (B)
- new net: J10.2 (Pin_2), JP24.1 (A)
- new net: J10.4 (Pin_4), JP22.1 (A)
- new net: J10.5 (Pin_5), JP26.1 (A), JP27.2 (B)
- new net: J9.1 (Pin_1), OA2.2 (-), OA2.6
- new net: J7.S, JP12.1 (A)
- new net: J3.1 (Pin_1), JP17.2 (B)
- new net: J3.3 (Pin_3), JP15.2 (B)
- new net: J7.R, JP8.1 (A)
- new net +3.3V: C2.1, J2.5 (Pin_5), JP19.1 (A), JP21.1 (A), JP27.1 (A), JP7.1 (A), U1.21 (3V3), U2.8 (VCC)
- new net +5V: C1.1, J2.1 (Pin_1), JP18.2 (B), JP20.2 (B), JP26.2 (B), JP6.2 (B), U1.23 (5V)
- new net GND: C1.2, C2.2, C3.2, C4.2, J2.3 (Pin_3), J6.2, J8.2 (Pin_2), J9.2 (Pin_2), JP12.2 (B), JP13.2 (B), OA1.4 (V-), OA2.4 (V-), U1.22 (GND), U1.33 (GND), U2.4 (GND)
Other:
- note added: "a soic 8 for eeprom"
